File: lauflicht_charlie/lauflicht_charlie.sch (KiCad schematic (older format))
At the start: 9 parts

Commit message: fix LED numbers to match code
Parts:
- D?: value LED3 -> LED4
- D?: value LED4 -> LED3
Other:
- moved on the sheet: IC?
Changed lines of the file:
@@
-EESchema Schematic File Version 2  date Mo 06 Mai 2013 22:08:20 CEST
+EESchema Schematic File Version 2  date So 19 Mai 2013 21:49:01 CEST
 LIBS:power
 LIBS:device
@@
 Sheet 1 1
 Title ""
-Date "6 may 2013"
+Date "19 may 2013"
 Rev ""
 Comp ""
@@
 P 5050 3300
 F 0 "D?" H 5050 3400 50  0000 C CNN
-F 1 "LED4" H 5050 3200 50  0000 C CNN
+F 1 "LED3" H 5050 3200 50  0000 C CNN
 	1    5050 3300
 	0    -1   -1   0
@@
 P 4700 3300
 F 0 "D?" H 4700 3400 50  0000 C CNN
-F 1 "LED3" H 4700 3200 50  0000 C CNN
+F 1 "LED4" H 4700 3200 50  0000 C CNN
 	1    4700 3300
 	0    1    1    0
@@
 L ATMEGA16-P IC?
 U 1 1 5186B473
-P 2450 4350
-F 0 "IC?" H 1650 6080 50  0000 L BNN
-F 1 "ATMEGA16-P" H 2675 2350 50  0000 L BNN
-F 2 "DIL40" H 2950 2275 50  0001 C CNN
-	1    2450 4350
+P 2450 3750
+F 0 "IC?" H 1650 5480 50  0000 L BNN
+F 1 "ATMEGA16-P" H 2675 1750 50  0000 L BNN
+F 2 "DIL40" H 2950 1675 50  0001 C CNN
+	1    2450 3750
 	1    0    0    -1
 $EndComp
